File: Electronics/Sparki_Mainboard.sch (EAGLE design)
At the start: 92 parts, among them IC1 74595, IC2 74595, J1 1X2-3.5MM, U2 ATMEGA32U4-AU, U3 LP2985-33DBVR, U4 MMA8452Q, U5 NRF24L01SMD, X1 USBSMD, X3 05-JST-B5B-XH-A, X4 05-XH-JST-B5B-XH-A, X5 05-JST-B5B-XH-A, Y1 ANTENNA2SMD5

Commit message: Updated connectors, sensor multiplexing
Parts:
- removed BLUETOOTH: Bluetooth, arcbotics:M04SMD3
- removed C17: 10uF, SparkFun-Capacitors:CAP0603-CAP
- removed C18: 0.1uF, SparkFun-Capacitors:0.1UF-25V(+80/-20%)(0603)
- removed C19, C20: 8pf, SparkFun:CAP0402
- removed C21: 33nF, SparkFun:CAP0402
- removed C22: 2.2nF, SparkFun:CAP0402
- removed C23: 4.7pF, SparkFun:CAP0402
- removed C24: 1.0pF, SparkFun:CAP0402
- removed C25: 1.5pF, SparkFun:CAP0402
- removed L1: 3.9nH, SparkFun:INDUCTOR0402
- removed L2: 2.7nH, SparkFun:INDUCTOR0402
- removed L3: 8.2nH, SparkFun:INDUCTOR0402
- removed R16: 1M, SparkFun:RESISTOR0402
- removed R17: 22K, SparkFun:RESISTOR0402
- removed U$9: M04X2, SparkFun-Connectors:M04X2
- removed U5: NRF24L01SMD, SparkFun:NRF24L01SMD
- removed X6: (no value), adafruit:XTALNX5032
- removed Y1: ANTENNA2SMD5, SparkFun:ANTENNA2SMD5
- added R18, R19: 100, SparkFun-Passives:RESISTOR0603-RES
- added U$10: M08X2SMD, arcbotics:M08X2SMD
- JP2: value M102MMSMD -> M10; device SparkFun-Connectors:M102MMSMD -> arcbotics:M10
- R11, R12, R13: value 10k -> 47k
Connections:
- net LINE_MID renamed LINE_CENTER
- net PD5 renamed N$13
- removed net ANT: C24.2, C25.2, Y1.SIGNAL
- removed net N$20: C19.1, R16.1, U5.XC2, X6.P$2
- removed net N$23: C20.1, R16.2, U5.XC1, X6.P$1
- removed net N$24: L1.1, L3.2, U5.ANT2
- removed net N$25: C22.1, C23.1, L2.1, U5.VDD_PA
- removed net N$27: R17.1, U5.IREF
- removed net N$28: C21.1, U5.DVDD
- removed net N$33: L2.2, L3.1, U5.ANT1
- removed net N$34: C25.1, L1.2
- net GND: now also R19.2, U$10.10, U$10.5, U$10.6, U$6.VEE; no longer BLUETOOTH.2, C17.2, C18.2, C19.2, C20.2, C21.2, C22.2, C23.2, C24.1, R17.2, U$9.1, U5.VSS@0, U5.VSS@14, U5.VSS@17, U5.VSS@20, U5.VSS@8
- net MISO: now also U$10.16; no longer U$9.7, U5.MISO
- net MOSI: now also U$10.13; no longer U$9.6, U5.MOSI
- net PB4: now also U$10.15; no longer U$9.8, U5.IRQ
- net PB6: now also R18.2, R19.1, SONIC.2; no longer SONIC.3
- net PC6: now also SONIC.3; no longer SONIC.2
- net PD0: now also U$10.3
- net PD1: now also U$10.1
- net PF6: now also U$10.11; no longer U$9.3, U5.CE
- net PF7: now also U$10.12; no longer U$9.4, U5.CSN
- net RX: now also U$10.4; no longer BLUETOOTH.4
- net SCK: now also U$10.14; no longer U$9.5, U5.SCK
- net TX: now also U$10.2; no longer BLUETOOTH.3
- net VCC: now also U$10.7, U$10.8; no longer BLUETOOTH.1, JP2.3, U$6.VEE
- net VCC_3V3: now also JP2.3, U$10.9; no longer C17.1, C18.1, U$9.2, U5.VDD@15, U5.VDD@18, U5.VDD@7
- net V_BATT_POWER: now also R18.1
Other:
- moved on the sheet: SONIC
